File: 01_top/aliceball.kicad_pcb (KiCad board)
At the start: 2 copper layers, 314.4 x 98.8 mm, 64 parts, among them J1 Conn_01x01, J10 Conn_01x01, J11 Conn_01x01, J12 Conn_01x01, J13 Conn_01x01, J14 Conn_01x01, J15 Conn_01x01, J16 Conn_01x01, J2 Conn_01x01, J3 Conn_01x01, J4 Conn_01x01, J5 Conn_01x01, J6 Conn_01x01, J7 Conn_01x01, J8 Conn_01x01, J9 Conn_01x01, SW1 SW_PUSH, SW10 SW_PUSH, SW11 SW_PUSH, SW12 SW_PUSH, SW13 SW_PUSH, SW14 SW_PUSH, SW15 SW_PUSH, SW16 KEY_SWITCH, SW17 SW_PUSH, SW18 SW_PUSH, SW19 SW_PUSH, SW2 KEY_SWITCH, SW20 SW_PUSH, SW21 SW_PUSH, SW22 SW_PUSH, SW23 SW_PUSH, SW24 SW_PUSH, SW25 SW_PUSH, SW26 SW_PUSH, SW27 SW_PUSH, SW28 SW_PUSH, SW29 SW_PUSH, SW3 SW_PUSH, SW30 SW_PUSH, SW31 SW_PUSH, SW32 SW_PUSH, SW33 KEY_SWITCH, SW34 SW_PUSH, SW35 SW_PUSH, SW36 SW_PUSH, SW37 SW_PUSH, SW38 SW_PUSH, SW39 SW_PUSH, SW4 SW_PUSH, SW40 SW_PUSH, SW41 SW_PUSH, SW42 SW_PUSH, SW43 SW_PUSH, SW44 SW_PUSH, SW45 SW_PUSH, SW46 SW_PUSH, SW47 SW_PUSH, SW48 SW_PUSH, SW5 SW_PUSH, SW6 SW_PUSH, SW7 SW_PUSH, SW8 SW_PUSH, SW9 SW_PUSH

Commit message: rev 0.2
Parts:
- SW12: footprint kbd_SW_Hole:SW_Hole_1 -> kbd_SW_Hole:SW_Hole_1.25u
- SW16: footprint kbd_SW_Hole:SW_Hole_2 -> kbd_SW_Hole:SW_Hole_1.75u
- SW33: footprint kbd_SW_Hole:SW_Hole_2 -> kbd_SW_Hole:SW_Hole_1.5u
- SW40: footprint kbd_SW_Hole:SW_Hole_1 -> kbd_SW_Hole:SW_Hole_1.5u
- moved SW40 4.74 mm to (267.3, 89.6)
- moved SW33 4.74 mm to (239.1, 94.5)
- moved SW16 2.37 mm to (111.0, 94.2)
- moved SW12 2.36 mm to (82.9, 89.2)
- moved SW3 0.09 mm to (35.7, 68.1)
