File: 02_Assemble/aliceball.kicad_pcb (KiCad board)
At the start: 2 copper layers, 304.4 x 98.8 mm, 176 parts, among them J1 Conn_01x02, J18 Conn_02x04_Odd_Even, SW1 SW_PUSH, SW10 SW_PUSH, SW11 SW_PUSH, SW12 SW_PUSH, SW13 SW_PUSH, SW14 SW_PUSH, SW15 SW_PUSH, SW16 SW_PUSH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

Commit message: rev 0.2
Parts:
- J18: moved to B.Cu
- turned J18 to 180 degrees
Routing:
- net GND: track 1715.2 -> 1687.8 mm, vias 61 -> 60
- net VCC: track 1914.2 -> 1891.3 mm
- net unconnected-(J18-Pad5): track 0.00 -> 0.50 mm
