File: 02_Assemble_bmp/aliceball.kicad_pcb (KiCad board)
At the start: 2 copper layers, 304.4 x 98.8 mm, 176 parts, among them J1 Conn_01x02, J18 Conn_02x04_Odd_Even, SW1 SW_PUSH, SW10 SW_PUSH, SW11 SW_PUSH, SW12 SW_PUSH, SW13 SW_PUSH, SW14 SW_PUSH, SW15 SW_PUSH, SW16 SW_PUSH, SW17 SW_PUSH, SW18 SW_PUSH, SW19 SW_PUSH, SW2 SW_PUSH, SW20 SW_PUSH, SW21 SW_PUSH, SW22 SW_PUSH, SW23 SW_PUSH, SW24 SW_PUSH, SW24_2 SW_PUSH, SW25 RotaryEncoder_Switch, SW26 SW_PUSH, SW27 SW_PUSH, SW28 SW_PUSH, SW29 SW_PUSH, SW3 SW_PUSH, SW30 SW_PUSH, SW31 SW_PUSH, SW32 SW_PUSH, SW33 SW_PUSH, SW34 SW_PUSH, SW35 SW_PUSH, SW36 SW_PUSH, SW37 SW_PUSH, SW38 SW_PUSH, SW39 SW_PUSH, SW4 SW_PUSH, SW40 SW_PUSH, SW41 SW_PUSH, SW42 SW_PUSH, SW43 SW_PUSH, SW44 SW_PUSH, SW45 SW_PUSH, SW46 SW_PUSH, SW47 SW_PUSH, SW48 SW_PUSH, SW49 SW_PUSH, SW5 SW_PUSH, SW6 SW_PUSH, SW7 SW_PUSH, SW8 SW_PUSH, SW9 SW_PUSH, U1 BLEMicroPro

Commit message: add bmp version
Parts:
- moved J1 2.10 mm to (165.4, 22.7)
- moved D45 0.76 mm to (319.7, 34.1)
Connections:
- J18 pad 1: (no net) -> unconnected-(J18-Pad1)
- U1 pad 1: LED -> B1
- U1 pad 12: B1 -> CS
- U1 pad 13: CS -> LED
Routing:
- net B1: track 155.7 -> 124.3 mm, vias 6 -> 5
- net CS: track 185.6 -> 209.9 mm, vias 0 -> 2
- net LED: track 46.4 -> 26.0 mm, vias 2 -> 3
- net GND: track 1715.2 -> 1709.8 mm
- net Row0: track 338.3 -> 333.0 mm, vias 12 -> 13
- net Bat+: track 115.9 -> 114.0 mm
- net VCC: track 1914.2 -> 1915.8 mm

Commit message: rev 0.2
Parts:
- D1, D10, D11, D12, D13, D14, D15, D16, D17, D18, D19, D2, D20, D21, D22, D23, D24, D25, D26, D27, D28, D29, D3, D30, D31, D32, D33, D34, D35, D36, D37, D38, D39, D4, D40, D41, D42, D43, D44, D45, D46, D47, D48, D5, D6, D7, D8, D9: footprint kbd_Parts:Diode_TH_SMD -> kbd_Parts:Diode_SMD
- H1, H10, H11, H12, H13, H14, H15, H16, H2, H3, H4, H5, H6, H7, H8, H9: footprint MountingHole:MountingHole_2.2mm_M2 -> kbd_Hole:m2_Screw_Hole
- J18: value Conn_02x04_Odd_Even -> Conn_01x08; footprint kbd_Parts:ADNS-9800-module -> kbd_Parts:PMW3389_board
- L1, L10, L11, L12, L13, L14, L15, L16, L17, L18, L19, L2, L20, L21, L22, L23, L24, L25, L26, L27, L28, L29, L3, L30, L31, L32, L33, L34, L35, L36, L37, L38, L39, L4, L40, L41, L42, L43, L44, L45, L46, L47, L48, L49, L5, L50, L51, L52, L53, L54, L55, L56, L57, L58, L59, L6, L7, L8, L9: footprint kbd_Parts:LED_SK6812MINI-E_BL -> kbd_Parts:LED_SK6812MINI-E_BL_cut_silk
- SW1, SW10, SW11, SW13, SW14, SW15, SW17, SW18, SW19, SW20, SW21, SW22, SW23, SW24, SW26, SW27, SW28, SW29, SW30, SW31, SW32, SW34, SW35, SW36, SW37, SW38, SW39, SW4, SW42, SW43, SW44, SW46, SW47, SW48, SW5, SW6, SW7, SW8, SW9: footprint kbd_SW:CherryMX_Hotswap_1.0u -> kbd_SW:CherryMX_Hotswap_1u_no_silk
- SW12: footprint kbd_SW:CherryMX_Hotswap_1.0u -> kbd_SW:CherryMX_Hotswap_1.25u_no_silk
- SW16: footprint kbd_SW:CherryMX_Hotswap_2u_Rev -> kbd_SW:CherryMX_Hotswap_1.75u_no_silk
- SW2: footprint kbd_SW:CherryMX_Hotswap_1.25u -> kbd_SW:CherryMX_Hotswap_1.25u_no_silk
- SW3: footprint kbd_SW:CherryMX_Hotswap_1.75u -> kbd_SW:CherryMX_Hotswap_1.75u_no_silk
- SW33: footprint kbd_SW:CherryMX_Hotswap_2u_Rev -> kbd_SW:CherryMX_Hotswap_1.5u_no_silk
- SW40: footprint kbd_SW:CherryMX_Hotswap_1.0u -> kbd_SW:CherryMX_Hotswap_1.5u_no_silk
- SW41: footprint kbd_SW:CherryMX_Hotswap_1.0u_Small1 -> kbd_SW:CherryMX_Hotswap_1u_Small1_no_silk
- SW45: footprint kbd_SW:CherryMX_Hotswap_1.5u -> kbd_SW:CherryMX_Hotswap_1.5u_no_silk
- moved H8 44.2 mm to (154.1, 83.9)
- moved H6 32.0 mm to (197.9, 83.9)
- moved H7 31.0 mm to (176.0, 105.9)
- moved D24 5.98 mm to (163.4, 34.5)
- moved D33 5.90 mm to (247.8, 93.9)
- moved SW24_2 5.45 mm to (166.5, 34.7), turned to 90 degrees
- moved D12 5.18 mm to (92.2, 91.6)
- moved D40 5.13 mm to (276.6, 89.0)
- moved L12 4.76 mm to (268.0, 94.5)
- moved SW33 4.73 mm to (239.1, 94.5), turned to 10 degrees
- moved L19 4.71 mm to (239.8, 99.3)
- moved SW40 4.70 mm to (267.3, 89.6)
- moved D2 4.39 mm to (42.1, 49.9)
- moved D37 4.21 mm to (272.0, 31.2)
- moved D27 4.11 mm to (226.3, 58.7)
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Connections:
- J18 pad 1: unconnected-(J18-Pad1) -> VCC
- J18 pad 2: CS -> MISO
- J18 pad 3: GND -> MOSI
- J18 pad 4: MOSI -> SCLK
- J18 pad 5: unconnected-(J18-Pad5) -> CS
- J18 pad 6: SCLK -> unconnected-(J18-Pad6)
- J18 pad 7: VCC -> GND
- J18 pad 8: MISO -> unconnected-(J18-Pad8)
- U1 pad 17: Col3 -> Col0
- U1 pad 18: Col2 -> Col1
- U1 pad 19: Col1 -> Col2
- U1 pad 20: Col0 -> Col3
Routing:
- net Col0: track 432.8 -> 689.5 mm, vias 10 -> 8
- net Col1: track 427.3 -> 660.2 mm, vias 17 -> 15
- net Col3: track 386.5 -> 587.8 mm, vias 15 -> 21
- net VCC: track 1915.8 -> 1798.4 mm, vias 6 -> 0
- net Col4: track 329.8 -> 380.1 mm, vias 13 -> 22
- net Row3: track 400.9 -> 355.7 mm, vias 15 -> 7
- net Row2: track 394.1 -> 351.4 mm, vias 12 -> 3
- net Row0: track 333.0 -> 303.0 mm, vias 13 -> 6
- net Col5: track 355.3 -> 371.7 mm, vias 10 -> 18
- net CS: track 209.9 -> 193.5 mm, vias 2 -> 0
- net Net-(L33-Pad1): track 27.6 -> 41.9 mm
- net Row1: track 369.0 -> 355.3 mm, vias 16 -> 6
- net GND: track 1709.8 -> 1697.4 mm, vias 61 -> 66
- net Net-(L40-Pad1): track 24.3 -> 36.4 mm
- net Net-(L10-Pad1): track 18.8 -> 30.7 mm, vias 2 -> 4
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Other:
- outline, holes or cut-outs redrawn
- board text added: "aliceball_rev0.2"
- board text added: "for GL516 case"
- board text removed: "aliceball_rev0.1"
